Commit message: update description

File: ydpibot_description/urdf/ydpibot_description.urdf (robot description, URDF)
Before this commit: robot ydpibot_describtion, 13 links, 12 joints
Links:
- removed link dummy
- added link Lower_Base, mass 0.11353; collision mesh filename=package://ydpibot_description/meshes/Lower_Base.STL; visual mesh filename=package://ydpibot_description/meshes/Lower_Base.STL
- link Base_upper: geometry collision mesh filename=package://ydpibot_description/meshes/Base_upper.STL; visual mesh filename=package://ydpibot_description/meshes/Base_upper.STL
- link Caster Wheel: geometry collision mesh filename=package://ydpibot_description/meshes/Caster Wheel.STL; visual mesh filename=package://ydpibot_description/meshes/Caster Wheel.STL
- link Caster Wheel Base: geometry collision mesh filename=package://ydpibot_description/meshes/Caster Wheel Base.STL; visual mesh filename=package://ydpibot_description/meshes/Caster Wheel Base.STL
- link Caster Wheel cage: geometry collision mesh filename=package://ydpibot_description/meshes/Caster Wheel cage.STL; visual mesh filename=package://ydpibot_description/meshes/Caster Wheel cage.STL
- link Lidar: mass 0.032124 -> 0.0321236105023131; geometry collision mesh filename=package://ydpibot_description/meshes/Lidar.STL; visual mesh filename=package://ydpibot_description/meshes/Lidar.STL
- link Wheel1: mass 0.075104 -> 0.075103699374881; geometry collision mesh filename=package://ydpibot_description/meshes/Wheel1.STL; visual mesh filename=package://ydpibot_description/meshes/Wheel1.STL
- link Wheel2: geometry collision mesh filename=package://ydpibot_description/meshes/Wheel2.STL; visual mesh filename=package://ydpibot_description/meshes/Wheel2.STL
- link base_link: geometry collision mesh filename=package://ydpibot_description/meshes/base_link.STL; visual mesh filename=package://ydpibot_description/meshes/base_link.STL
- link spacer1: geometry collision mesh filename=package://ydpibot_description/meshes/spacer1.STL; visual mesh filename=package://ydpibot_description/meshes/spacer1.STL
- link spacer2: mass 0.0038202 -> 0.00382017666676519; geometry collision mesh filename=package://ydpibot_description/meshes/spacer2.STL; visual mesh filename=package://ydpibot_description/meshes/spacer2.STL
- link spacer3: mass 0.0038202 -> 0.00382017666676519; geometry collision mesh filename=package://ydpibot_description/meshes/spacer3.STL; visual mesh filename=package://ydpibot_description/meshes/spacer3.STL
- link spacer4: mass 0.0038202 -> 0.00382017666676519; geometry collision mesh filename=package://ydpibot_description/meshes/spacer4.STL; visual mesh filename=package://ydpibot_description/meshes/spacer4.STL
Joints:
- removed joint dummy_joint
- added joint Lower_Base_joint: type fixed, parent base_link, child Lower_Base, origin xyz=0.10092 -0.17099 0.099422 rpy=1.5708 0 0, axis 0 0 0
- joint spacer4_joint: origin xyz=-0.0846153846153846 0 0.0549999999999999 rpy=0 0.147154651933592 0 -> xyz=-0.084615 0 0.055 rpy=0 0.14715 0

Commit message: perfect description

File: ydpibot_description/urdf/ydpibot_description.urdf (robot description, URDF)
Before this commit: robot ydpibot_description, 13 links, 12 joints
Links:
- removed link Base_upper
- removed link Caster Wheel
- removed link Caster Wheel Base
- removed link Caster Wheel cage
- removed link Lidar
- removed link Lower_Base
- removed link Wheel1
- removed link Wheel2
- added link Upper_base, mass 0.072243; collision mesh filename=package://ydpibot_description/meshes/Upper_base.STL; visual mesh filename=package://ydpibot_description/meshes/Upper_base.STL
- added link base_scan, mass 0.032124; collision mesh filename=package://ydpibot_description/meshes/base_scan.STL; visual mesh filename=package://ydpibot_description/meshes/base_scan.STL
- added link caster_wheel, mass 0.017472; collision mesh filename=package://ydpibot_description/meshes/caster_wheel.STL; visual mesh filename=package://ydpibot_description/meshes/caster_wheel.STL
- added link caster_wheel_base, mass 0; collision mesh filename=package://ydpibot_description/meshes/caster_wheel_base.STL; visual mesh filename=package://ydpibot_description/meshes/caster_wheel_base.STL
- added link caster_wheel_cage, mass 0.056621; collision mesh filename=package://ydpibot_description/meshes/caster_wheel_cage.STL; visual mesh filename=package://ydpibot_description/meshes/caster_wheel_cage.STL
- added link left_wheel, mass 0.075104; collision mesh filename=package://ydpibot_description/meshes/left_wheel.STL; visual mesh filename=package://ydpibot_description/meshes/left_wheel.STL
- added link right_wheel, mass 0.075104; collision mesh filename=package://ydpibot_description/meshes/right_wheel.STL; visual mesh filename=package://ydpibot_description/meshes/right_wheel.STL
- link spacer2: mass 0.00382017666676519 -> 0.0038202
- link spacer3: mass 0.00382017666676519 -> 0.0038202
- link spacer4: mass 0.00382017666676519 -> 0.0038202
Joints:
- removed joint Base_upper_joint
- removed joint Caster Wheel Base_joint
- removed joint Caster Wheel cage_joint
- removed joint Caster Wheel_joint
- removed joint Lidar_joint
- removed joint Lower_Base_joint
- removed joint Wheel1_joint
- removed joint Wheel2_joint
- removed joint spacer3_joint
- added joint Upper_base: type fixed, parent base_link, child Upper_base, origin xyz=-0.0019675 0 0.0895 rpy=0 0 0, axis 0 0 0
- added joint base_scan_joint: type fixed, parent Upper_base, child base_scan, origin xyz=-0.0397250065539057 0 0.049480432620002 rpy=0 0 0, axis 0 0 0
- added joint caster_wheel_base_joint: type fixed, parent base_link, child caster_wheel_base, origin xyz=0.0550228988474612 -0.0125000000000001 0.0464999999999998 rpy=0 0 0, axis 0 0 0
- added joint caster_wheel_cage_joint: type fixed, parent caster_wheel_base, child caster_wheel_cage, origin xyz=-0.00235708009540958 0.00411504444057814 -0.00400000000000002 rpy=0 0 0, axis 0 0 0
- added joint caster_wheel_joint: type fixed, parent caster_wheel_cage, child caster_wheel, origin xyz=0.0350067859440261 0.00481885237829768 -0.0229999999999999 rpy=0 0 0, axis 0 0 0
- added joint left_wheel_joint: type continuous, parent base_link, child left_wheel, origin xyz=-0.021967 0.08 0.0325 rpy=0 0 0, axis 0 -1 0
- added joint right_wheel_joint: type continuous, parent base_link, child right_wheel, origin xyz=-0.021967 -0.055 0.0325 rpy=0 0 0, axis 0 -1 0
- added joint spacer3_joiint: type continuous, parent Upper_base, child spacer3, origin xyz=-0.0846153846153847 -0.0549999999999999 0 rpy=0 0 0, axis 0 0 1
- joint spacer1_joint: axis 0 1 0 -> 0 0 1; origin xyz=0.084615 0 -0.055 rpy=0 0.33559 0 -> xyz=0.084615 0.055 0 rpy=0 0 0; parent Base_upper -> Upper_base
- joint spacer2_joint: axis 0 1 0 -> 0 0 1; origin xyz=0.084615 0 0.055 rpy=0 0.33674 0 -> xyz=0.0846153846153847 -0.0549999999999999 0 rpy=0 0 0; parent Base_upper -> Upper_base
- joint spacer4_joint: axis 0 1 0 -> 0 0 1; origin xyz=-0.084615 0 0.055 rpy=0 0.14715 0 -> xyz=-0.0846153846153847 0.055 0 rpy=0 0 0; parent Base_upper -> Upper_base

Commit message: gazebo+rviz updated

File: ydpibot_description/urdf/ydpibot_description.urdf (robot description, URDF)
Before this commit: robot ydpibot_description, 12 links, 11 joints
Joints:
- joint left_wheel_joint: axis 0 -1 0 -> 0 1 0
- joint right_wheel_joint: axis 0 -1 0 -> 0 1 0

Commit message: sim

File: ydpibot_description/urdf/ydpibot_description.urdf (robot description, URDF)
Before this commit: robot ydpibot_description, 12 links, 11 joints
Links:
- removed link caster_wheel
- removed link caster_wheel_base
- removed link caster_wheel_cage
- added link IMU, mass 0.00046193; collision mesh filename=package://ydpibot_description/meshes/IMU.STL; visual mesh filename=package://ydpibot_description/meshes/IMU.STL
- added link caster_wheel_, mass 0.12787; collision mesh filename=package://ydpibot_description/meshes/caster_wheel_.STL; visual mesh filename=package://ydpibot_description/meshes/caster_wheel_.STL
Joints:
- removed joint caster_wheel_base_joint
- removed joint caster_wheel_cage_joint
- removed joint caster_wheel_joint
- added joint IMU_joint: type fixed, parent base_link, child IMU, origin xyz=0.000205 0 0.04234 rpy=1.5708 0 0, axis 0 0 -1
- added joint caster_wheel__joint: type fixed, parent base_link, child caster_wheel_, origin xyz=0.069075 0 0.033565 rpy=-3.1416 0 0, axis 0 0 -1
- joint base_scan_joint: axis 0 0 0 -> 0 0 -1; origin xyz=-0.0397250065539057 0 0.049480432620002 rpy=0 0 0 -> xyz=-0.039725 0 0.04948 rpy=0 0 0
- joint spacer2_joint: origin xyz=0.0846153846153847 -0.0549999999999999 0 rpy=0 0 0 -> xyz=0.084615 -0.055 0 rpy=0 0 0
- joint spacer3_joiint: origin xyz=-0.0846153846153847 -0.0549999999999999 0 rpy=0 0 0 -> xyz=-0.084615 -0.055 0 rpy=0 0 0
- joint spacer4_joint: origin xyz=-0.0846153846153847 0.055 0 rpy=0 0 0 -> xyz=-0.084615 0.055 0 rpy=0 0 0

Commit message: slam

File: ydpibot_description/urdf/ydpibot_description.urdf (robot description, URDF)
Before this commit: robot ydpibot_description, 11 links, 10 joints
Links:
- link IMU: mass 0.00046193 -> 0.0014392
- link base_link: mass 0.11353 -> 1.11353
- link caster_wheel_: mass 0.12787 -> 0.4
- link left_wheel: mass 0.075104 -> 0.1
- link right_wheel: mass 0.075104 -> 0.1
- link spacer1: mass 0.0038202 -> 0.0049983
- link spacer2: mass 0.0038202 -> 0.0049983
- link spacer3: mass 0.0038202 -> 0.0049983
- link spacer4: mass 0.0038202 -> 0.0049983
Joints:
- joint IMU_joint: axis 0 0 -1 -> 0 0 0
- joint base_scan_joint: axis 0 0 -1 -> 0 0 0
- joint caster_wheel__joint: axis 0 0 -1 -> 0 0 0
- joint spacer1_joint: axis 0 0 1 -> 0 0 0; type continuous -> fixed
- joint spacer2_joint: axis 0 0 1 -> 0 0 0; type continuous -> fixed
- joint spacer3_joiint: axis 0 0 1 -> 0 0 0; type continuous -> fixed
- joint spacer4_joint: axis 0 0 1 -> 0 0 0; type continuous -> fixed

Commit message: rviz mapping file

File: ydpibot_description/urdf/ydpibot_description.urdf (robot description, URDF)
Before this commit: robot ydpibot_description, 11 links, 10 joints
Links:
- link base_link: mass 1.11353 -> None

Commit message: sim-map

File: ydpibot_description/urdf/ydpibot_description.urdf (robot description, URDF)
Before this commit: robot ydpibot_description, 11 links, 10 joints
Links:
- link base_link: mass None -> 1.11353

Commit message: edit urdf

File: ydpibot_description/urdf/ydpibot_description.urdf (robot description, URDF)
Before this commit: robot ydpibot_description, 11 links, 10 joints
Links:
- added link base_footprint
Joints:
- added joint base_footprint: type fixed, parent base_link, child base_footprint, origin xyz=0 0 0 rpy=0 0 0, axis 0 0 0
- joint base_scan_joint: origin xyz=-0.039725 0 0.04948 rpy=0 0 0 -> xyz=-0.039725 0 0.13948 rpy=0 0 0; parent Upper_base -> base_footprint
